File: CAD files/PCB/hot shoe IMU tracker.kicad_sch (KiCad schematic)
At the start: 23 parts, among them J1 USB_B_Micro, J2 Micro_SD_Card, J3 OLED, J4 BNO085, Q1 2N7002, SW1 Power, SW2 Start, SW3 Stop, U1 ESP32-C3_SUPERMINI_TH, U2 TP4056-42-ESOP8

Commit message: Add files via upload
Parts:
- BT1: MPN (none) -> B2B-ZR-SM4-TF
- C1: MPN (none) -> GRM155R71C104KA88D
- C2: MPN (none) -> GRM155R61A106ME11D
- D1: MPN (none) -> LTST-C171KGKT
- D2: MPN (none) -> LTST-C170KRKT
- J1: MPN (none) -> 0475900001
- J2: MPN (none) -> 1040310811
- J3, J4: MPN (none) -> SSM-104-L-SV-K-TR
- Q1: MPN (none) -> 2N7002
- R1, R2: MPN (none) -> CRCW08051K00FKEA
- R3: MPN (none) -> RCWP0575400RGKS6
- R4: MPN (none) -> CRCW08051K20FKEA
- R5, R6, R7, R8: MPN (none) -> CRCW080510K0FKEA
- SW1, SW2, SW3: MPN (none) -> RS-282G05A3-SM RT
- U1: MPN (none) -> 26892
- U2: MPN (none) -> TPB4056A20-ES1R
Changed lines of the file:
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@@
+			)
+		)
+		(property "MPN" "TPB4056A20-ES1R"
+			(at 60.96 40.64 0)
+			(effects
+				(font
+					(size 1.27 1.27)
+				)
+				(hide yes)
 			)
 		)
@@
 			)
 		)
+		(property "MPN" "CRCW080510K0FKEA"
+			(at 140.97 96.52 0)
+			(effects
+				(font
+					(size 1.27 1.27)
+				)
+				(hide yes)
+			)
+		)
 		(pin "1"
 		)
@@
 			)
 		)
+		(property "MPN" "CRCW08051K20FKEA"
+			(at 73.66 50.8 0)
+			(effects
+				(font
+					(size 1.27 1.27)
+				)
+				(hide yes)
+			)
+		)
 		(pin "1"
 		)
@@
 			)
 		)
+		(property "MPN" "0475900001"
+			(at 88.9 17.78 90)
+			(effects
+				(font
+					(size 1.27 1.27)
+				)
+				(hide yes)
+			)
+		)
 		(pin "4"
 		)
@@
 			)
 		)
+		(property "MPN" "RS-282G05A3-SM RT"
+			(at 130.81 107.95 0)
+			(effects
+				(font
+					(size 1.27 1.27)
+				)
+				(hide yes)
+			)
+		)
 		(pin "2"
 		)
@@
 			)
 		)
+		(property "MPN" "26892"
+			(at 179.07 35.56 0)
+			(effects
+				(font
+					(size 1.27 1.27)
+				)
+				(hide yes)
+			)
+		)
 		(pin "3.3"
 		)
@@
 			)
 		)
+		(property "MPN" "1040310811"
+			(at 247.65 58.42 0)
+			(effects
+				(font
+					(size 1.27 1.27)
+				)
+				(hide yes)
+			)
+		)
 		(pin "4"
 		)
@@
 			)
 		)
+		(property "MPN" "SSM-104-L-SV-K-TR"
+			(at 229.87 35.56 0)
+			(effects
+				(font
+					(size 1.27 1.27)
+				)
+				(hide yes)
+			)
+		)
 		(pin "4"
 		)
@@
 			)
 		)
+		(property "MPN" "B2B-ZR-SM4-TF"
+			(at 86.36 40.64 0)
+			(effects
+				(font
+					(size 1.27 1.27)
+				)
+				(hide yes)
+			)
+		)
 		(pin "2"
 		)
@@
 			)
 		)
+		(property "MPN" "SSM-104-L-SV-K-TR"
+			(at 104.14 54.61 90)
+			(effects
+				(font
+					(size 1.27 1.27)
+				)
+				(hide yes)
+			)
+		)
 		(pin "10"
 		)
@@
 			)
 		)
+		(property "MPN" "CRCW080510K0FKEA"
+			(at 125.73 96.52 0)
+			(effects
+				(font
+					(size 1.27 1.27)
+				)
+				(hide yes)
+			)
+		)
 		(pin "1"
 		)
@@
 			)
 		)
+		(property "MPN" "GRM155R61A106ME11D"
+			(at 222.25 73.66 0)
+			(effects
+				(font
+					(size 1.27 1.27)
+				)
+				(hide yes)
+			)
+		)
 		(pin "2"
 		)
@@
 			)
 		)
+		(property "MPN" "2N7002"
+			(at 140.97 50.8 90)
+			(effects
+				(font
+					(size 1.27 1.27)
+				)
+				(hide yes)
+			)
+		)
 		(pin "3"
 		)
@@
 			)
 		)
+		(property "MPN" "RCWP0575400RGKS6"
+			(at 60.96 22.86 0)
+			(effects
+				(font
+					(size 1.27 1.27)
+				)
+				(hide yes)
+			)
+		)
 		(pin "2"
 		)
@@
 			)
 		)
+		(property "MPN" "RS-282G05A3-SM RT"
+			(at 116.84 107.95 0)
+			(effects
+				(font
+					(size 1.27 1.27)
+				)
+				(hide yes)
+			)
+		)
 		(pin "2"
 		)
@@
 			)
 		)
+		(property "MPN" "LTST-C170KRKT"
+			(at 41.91 26.67 90)
+			(effects
+				(font
+					(size 1.27 1.27)
+				)
+				(hide yes)
+			)
+		)
 		(pin "2"
 		)
@@
 			)
 		)
+		(property "MPN" "CRCW08051K00FKEA"
+			(at 35.56 36.83 0)
+			(effects
+				(font
+					(size 1.27 1.27)
+				)
+				(hide yes)
+			)
+		)
 		(pin "1"
 		)
@@
 			)
 		)
+		(property "MPN" "LTST-C171KGKT"
+			(at 35.56 26.67 90)
+			(effects
+				(font
+					(size 1.27 1.27)
+				)
+				(hide yes)
+			)
+		)
 		(pin "2"
 		)
@@
 			)
 		)
+		(property "MPN" "CRCW080510K0FKEA"
+			(at 220.98 46.99 0)
+			(effects
+				(font
+					(size 1.27 1.27)
+				)
+				(hide yes)
+			)
+		)
 		(pin "1"
 		)
@@
 			)
 		)
+		(property "MPN" "GRM155R71C104KA88D"
+			(at 223.52 25.4 0)
+			(effects
+				(font
+					(size 1.27 1.27)
+				)
+				(hide yes)
+			)
+		)
 		(pin "2"
 		)
@@
 			)
 		)
+		(property "MPN" "CRCW08051K00FKEA"
+			(at 41.91 36.83 0)
+			(effects
+				(font
+					(size 1.27 1.27)
+				)
+				(hide yes)
+			)
+		)
 		(pin "1"
 		)
@@
 			)
 		)
+		(property "MPN" "RS-282G05A3-SM RT"
+			(at 146.05 107.95 0)
+			(effects
+				(font
+					(size 1.27 1.27)
+				)
+				(hide yes)
+			)
+		)
 		(pin "2"
 		)
@@
 			(at 111.76 96.52 0)
 			(effects
+				(font
+					(size 1.27 1.27)
+				)
+				(hide yes)
+			)
+		)
+		(property "MPN" "CRCW080510K0FKEA"
+			(at 111.76 96.52 0)
+			(effects
